File: Kicad_proj/STM32H743_board_wfl/04_bmi088_imu_sensor.kicad_sch (KiCad schematic)
At the start: 0 parts

Commit message: schematic filenames update
Other:
- company: (none) -> by wojtron
- title: (none) -> STM32H743 board IMU BMI088 schematics
Changed lines of the file:
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@@
 	(generator_version "10.0")
 	(paper "A4")
+	(title_block
+		(title "STM32H743 board IMU BMI088 schematics")
+		(company "by wojtron")
+	)
 )

Commit message: v0.3 uzupelniony prebom + placement BMI088 na sch
Parts:
- added U4: BMI088, Package_LGA:Bosch_LGA-16_4.5x3mm_P0.5mm_LayoutBorder7x1y_ClockwisePinNumbering, symbol Sensor_Motion:BMI088
Connections:
- new net: U4.2 (GNDA), U4.4 (GNDA)
Changed lines of the file:
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@@
 		(company "by wojtron")
 	)
+	(symbol
+		(lib_id "Sensor_Motion:BMI088")
+		(at 141.732 88.9 0)
+		(unit 1)
+		(body_style 1)
+		(exclude_from_sim no)
+		(in_bom yes)
+		(on_board yes)
+		(in_pos_files yes)
+		(dnp no)
+		(fields_autoplaced yes)
+		(property "Reference" "U4"
+			(at 146.4153 71.12 0)
+			(show_name no)
+			(do_not_autoplace no)
+			(effects
+				(font
+					(size 1.27 1.27)
+				)
+				(justify left)
+			)
+		)
+		(property "Value" "BMI088"
+			(at 146.4153 73.66 0)
+			(show_name no)
+			(do_not_autoplace no)
+			(effects
+				(font
+					(size 1.27 1.27)
+				)
+				(justify left)
+			)
+		)
+		(property "Footprint" "Package_LGA:Bosch_LGA-16_4.5x3mm_P0.5mm_LayoutBorder7x1y_ClockwisePinNumbering"
+			(at 125.222 90.17 0)
+			(hide yes)
+			(show_name no)
+			(do_not_autoplace no)
+			(effects
+				(font
+					(size 1.27 1.27)
+				)
+			)
+		)
+		(property "Datasheet" "https://www.bosch-sensortec.com/media/boschsensortec/downloads/datasheets/bst-bmi088-ds001.pdf"
+			(at 125.222 90.17 0)
+			(hide yes)
+			(show_name no)
+			(do_not_autoplace no)
+			(effects
+				(font
+					(size 1.27 1.27)
+				)
+			)
+		)
+		(property "Description" "Accelerometer, Gyroscope, 6-Axis Sensor, I2C / SPI interface, LGA-16"
+			(at 141.732 88.9 0)
+			(hide yes)
+			(show_name no)
+			(do_not_autoplace no)
+			(effects
+				(font
+					(size 1.27 1.27)
+				)
+			)
+		)
+		(pin "16"
+		)
+		(pin "15"
+		)
+		(pin "7"
+		)
+		(pin "8"
+		)
+		(pin "3"
+		)
+		(pin "12"
+		)
+		(pin "1"
+		)
+		(pin "5"
+		)
+		(pin "4"
+		)
+		(pin "2"
+		)
+		(pin "6"
+		)
+		(pin "9"
+		)
+		(pin "13"
+		)
+		(pin "14"
+		)
+		(pin "10"
+		)
+		(pin "11"
+		)
+		(instances
+			(project "STM32H743_board_wfl"
+				(path "/3ffbaf01-8fe7-4f96-b685-21b9df9d548a/ee56b707-46e2-4c51-8896-bad1360062d7"
+					(reference "U4")
+					(unit 1)
+				)
+			)
+		)
+	)
 )

Commit message: v.04d IMU
Parts:
- removed U4: BMI088, Package_LGA:Bosch_LGA-16_4.5x3mm_P0.5mm_LayoutBorder7x1y_ClockwisePinNumbering, symbol Sensor_Motion:BMI088
- added C27: 1uF, Capacitor_SMD:C_0603_1608Metric, symbol Device:C
- added C28, C29: 100nF, Capacitor_SMD:C_0402_1005Metric, symbol Device:C
- added L3: BLM21PG221SN1D, Inductor_SMD:L_0805_2012Metric, symbol Device:L_Ferrite
- added U5: BMI088, Package_LGA:Bosch_LGA-16_4.5x3mm_P0.5mm_LayoutBorder7x1y_ClockwisePinNumbering, symbol STM32H743_board_library_symbols:BMI088_
Connections:
- new net +3V3: L3.1
- new net +3V3_IMU: C27.1, C28.1, C29.1, L3.2, U5.11 (VDDIO), U5.3 (VDD)
- new net CS1_ACCELEROMETER: U5.14 (~{CSB1})
- new net CS2_GYROSCOPE: U5.5 (~{CSB2})
- new net GND: C27.2, C28.2, C29.2, U5.2 (NC), U5.4 (GNDA), U5.6 (GNDIO), U5.7 (PS)
- new net INT1_ACCELEROMETER: U5.16 (INT1)
- new net INT3_GYROSCOPE: U5.12 (INT3)
- new net SPI1_MISO: U5.10 (SDO2), U5.15 (SDO1)
- new net SPI1_MOSI: U5.9 (SDI/SDA)
- new net SPI1_SCK: U5.8 (SCK/SCL)
- no-connect marks 0 -> 2
