File: Kicad_proj/STM32H743_board_wfl/STM32H743_board_wfl.kicad_pcb (KiCad board)
At the start: 4 copper layers, 38.5 x 38.5 mm, 64 parts, among them J1 GPS, J2 ESC, J3 UART, J4 Tag_Connect_6pin, U1 LT8609SEV#PBF, U2 AP7361C-33E, U3 STM32H743VITx, U4 W25Q512JVEIQ, U5 BMI088, Y1 TSX-3225_16.0000MF18X-AC0

Commit message: PCB v0.7 routing part4
Parts:
- moved C19 2.27 mm to (117.2, 128.3), turned to 180 degrees
- moved C29 1.74 mm to (122.9, 129.2)
- moved C30 1.45 mm to (125.3, 123.7)
- moved R10 1.36 mm to (116.5, 107.2)
- moved R11 1.36 mm to (115.1, 107.2)
- moved R9 1.36 mm to (117.8, 107.2)
- moved C31 1.36 mm to (125.9, 129.1)
- moved R12 1.35 mm to (113.8, 107.2)
- moved L3 1.06 mm to (122.9, 131.0), turned to 180 degrees
- moved U5 0.98 mm to (125.2, 126.3)
- moved C18 0.57 mm to (117.0, 126.8)
- moved L2 0.15 mm to (119.0, 130.0)
- moved R8 0.06 mm to (103.0, 119.3)
Routing:
- net GND: track 207.6 -> 304.8 mm, vias 20 -> 31
- net /03_STM32H743_schematic/UART1_RX: track 0.00 -> 53.4 mm, vias 0 -> 2
- net /03_STM32H743_schematic/UART1_TX: track 0.00 -> 52.5 mm, vias 0 -> 2
- net +3V3: track 57.7 -> 78.4 mm, vias 8 -> 12
- net /03_STM32H743_schematic/UART2_TX: track 0.00 -> 15.0 mm
- net Net-(C25-Pad1): track 4.07 -> 17.5 mm, vias 0 -> 2
- net /03_STM32H743_schematic/UART2_RX: track 0.00 -> 12.9 mm
- net INT3_GYROSCOPE: track 0.00 -> 12.7 mm, vias 0 -> 2
- net +3V3_IMU: track 0.00 -> 11.9 mm, vias 0 -> 1
- net SPI1_MISO: track 0.00 -> 10.9 mm, vias 0 -> 2
- net CS1_ACCELEROMETER: track 0.00 -> 10.8 mm, vias 0 -> 2
- net Net-(U3-VDDA): track 8.17 -> 18.5 mm
- net /03_STM32H743_schematic/TELEMETRY: track 0.00 -> 6.79 mm
- net SPI1_MOSI: track 0.00 -> 6.31 mm
- net SPI1_SCK: track 0.00 -> 6.05 mm
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